Commit message: Working project2

File: my_robot/urdf/my_robot.xacro (robot description, xacro)
@@ -11,5 +11,5 @@
     <pose>0 0 0.3 0 0 0</pose>
     <inertial>
-      <mass value="15.0"/>
+      <mass value="10.0"/>
       <origin xyz="0.0 0 0" rpy=" 0 0 0"/>
       <inertia
@@ -54,5 +54,5 @@
   <link name='right_wheel'>
     <inertial>
-      <mass value="5.0"/>
+      <mass value="2.0"/>
       <origin xyz="0 0 0" rpy=" 0 1.5707 1.5707"/>
       <inertia
@@ -85,5 +85,5 @@
   <link name='left_wheel'>
     <inertial>
-      <mass value="5.0"/>
+      <mass value="2.0"/>
       <origin xyz="0 0 0" rpy=" 0 1.5707 1.5707"/>
       <inertia
